File: hum_contr/hum_contr.kicad_pcb (KiCad board)
At the start: 2 copper layers, 70.4 x 38 mm, 22 parts, among them J3 Screw_Terminal_01x04, U1 ESP-12E, U10 HT7333, U2 BME680, U3 EL817, U4 EL817, U5 EL817, U6 EL817

Commit message: first commit
Parts:
- removed J3: Screw_Terminal_01x04, TerminalBlock_TE-Connectivity:TerminalBlock_TE_282834-4_1x04_P2.54mm_Horizontal
- removed U2: BME680, Package_LGA:Bosch_LGA-8_3x3mm_P0.8mm_ClockwisePinNumbering
Routing:
- net Net-(J3-Pin_4): track 16.5 -> 0.00 mm
- net Net-(J3-Pin_1): track 9.98 -> 0.00 mm
- net Net-(J3-Pin_3): track 9.72 -> 0.00 mm
- net Net-(J3-Pin_2): track 6.90 -> 0.00 mm
Other:
- board size 70.4 x 38 mm -> 45 x 38 mm
