File: hum_contr/hum_contr.kicad_sch (KiCad schematic)
At the start: 25 parts, among them J1 Sensor Power ON/OFF, J3 Screw_Terminal_01x04, U1 ESP-12E, U10 HT7333, U2 BME680, U3 EL817, U4 EL817, U5 EL817, U6 EL817, U7 EL817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

Commit message: first commit
Parts:
- removed J3: Screw_Terminal_01x04, TerminalBlock_TE-Connectivity:TerminalBlock_TE_282834-4_1x04_P2.54mm_Horizontal, symbol Connector:Screw_Terminal_01x04
- removed U2: BME680, Package_LGA:Bosch_LGA-8_3x3mm_P0.8mm_ClockwisePinNumbering, symbol Sensor:BME680
Other:
- company: (none) -> CYBEREX TECH
- title: (none) -> Контроллер управления увлажнителем
- moved on the sheet: C2, J1, J2, R1, R10, R11, R12, R2, R3, R4, R5, R6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
